File: v4/hardware/kicad/nlink-lite/nlink-lite.kicad_pcb (KiCad board)
At the start: 4 copper layers, 39 x 16 mm, 21 parts, among them J1 USB_MiniB_PLUG_to_calc, J4 PROG_PADS_TC2030, SW1 PWR_SW, U1 ESP32-C3-MINI-1-N4, U3 CP2102N-A02-GQFN24, U4 TLV62569DBV, U5 USBLC6-2SC6

Commit message: Updated v4 pcb
Parts:
- C6, R4, R5: moved to B.Cu
- J4: value PROG_PADS_TC2030 -> PROG_PADS_2x3_POGO; footprint Connector:Tag-Connect_TC2030-IDC-FP_2x03_P1.27mm_Vertical -> Connector_PinHeader_1.27mm:PinHeader_2x03_P1.27mm_Vertical_SMD; moved to B.Cu
- moved R6 16.3 mm to (70.5, 52.1)
- moved C5 15.8 mm to (70.8, 55.2), turned to 90 degrees
- moved C4 15.2 mm to (70.5, 58.5), turned to 90 degrees
- moved C6 14.8 mm to (76.0, 53.5)
- moved R4 14.8 mm to (74.0, 53.5)
- moved R5 14.8 mm to (78.0, 53.5)
- moved D1 14.4 mm to (70.8, 53.0)
- moved J4 9.62 mm to (76.5, 57.5)
- moved R2 6.70 mm to (66.0, 59.3)
- moved R3 6.70 mm to (68.0, 59.3)
- moved L1 5.60 mm to (70.4, 62.5), turned to 90 degrees
- moved J1 5.49 mm to (52.0, 62.6), turned to 180 degrees
- moved U4 5.32 mm to (66.7, 62.4)
- moved C1 4.81 mm to (66.5, 52.3)
- moved C2 4.81 mm to (68.5, 52.3)
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Routing:
- net GND: track 0.00 -> 117.5 mm, vias 0 -> 1
- net +3V3: track 0.00 -> 55.5 mm, vias 0 -> 4
- net VBUS: track 0.00 -> 23.0 mm
- net CALC_DP: track 0.00 -> 15.0 mm, vias 0 -> 1
- net UART_RX: track 0.00 -> 13.7 mm, vias 0 -> 2
- net UART_TX: track 0.00 -> 13.0 mm, vias 0 -> 2
- net STATUS_LED: track 0.00 -> 12.9 mm, vias 0 -> 2
- net CALC_DM: track 0.00 -> 12.8 mm, vias 0 -> 1
- net IO0: track 0.00 -> 12.1 mm, vias 0 -> 1
- net EN: track 0.00 -> 11.7 mm, vias 0 -> 1
- net CP_RSTn: track 0.00 -> 9.61 mm
- net USB_DP: track 0.00 -> 9.09 mm, vias 0 -> 1
- net USB_DM: track 0.00 -> 9.05 mm, vias 0 -> 1
- net VBUS_IN: track 0.00 -> 9.02 mm
- net SW_NODE: track 0.00 -> 5.61 mm
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- added copper zone on B.Cu, net GND
- added copper zone on F.Cu, net GND
Other:
- board size 39 x 16 mm -> 40 x 15 mm
- board text added: "2:GND 1:3V3"
- board text added: "4:IO0 3:EN"
- board text added: "6:D+ 5:D-"
- board text added: "ANTENNA"
- board text added: "D+"
- board text added: "D-"
- board text added: "G"
- board text added: "PROG"
- board text added: "V+"
- board text added: "nlink-lite"
- board text added: "nlink-lite v4"
- board text removed: "nlink-lite ~38x16 chat-only stealth (placement seed, unrouted)"

Commit message: Community caught bugs
Parts:
- added C7: 10u, Capacitor_SMD:C_0805_2012Metric, B.Cu at (82.4, 55.6)
- added R10: 10k, Resistor_SMD:R_0402_1005Metric, B.Cu at (78.0, 53.5)
- added R7: 10k, Resistor_SMD:R_0402_1005Metric, B.Cu at (74.3, 62.0)
- added R8: 470, Resistor_SMD:R_0402_1005Metric, F.Cu at (70.5, 52.1)
- added R9: 10k, Resistor_SMD:R_0402_1005Metric, B.Cu at (74.3, 60.8)
- C5: value 10u -> 100n; footprint Capacitor_SMD:C_0805_2012Metric -> Capacitor_SMD:C_0402_1005Metric; moved to B.Cu
- R1: value 10k -> 1k
- R2: value 453k -> 22.1k; moved to B.Cu
- R3: value 100k -> 47.5k; moved to B.Cu
- R4: value 10k -> 453k; moved to F.Cu
- R5: value 10k -> 100k; moved to F.Cu
- R6: value 470 -> 10k; moved to B.Cu
- moved R5 11.3 mm to (68.2, 59.3)
- moved R4 9.68 mm to (66.2, 59.3)
- moved C5 5.46 mm to (76.0, 53.5), turned to 0 degrees
- moved R3 5.05 mm to (63.0, 60.0)
- moved R2 5.04 mm to (61.0, 60.0)
- moved C6 4.63 mm to (80.6, 53.0)
- moved R6 3.79 mm to (74.0, 53.5)
Connections:
- C5 pad 1: +3V3 -> EN
- C6 pad 1: EN -> +3V3
- J1 pad 4: (no net) -> GND
- J4 pad 4: IO0 -> BOOT
- R2 pad 1: +3V3 -> VBUS
- R2 pad 2: FB_3V3 -> CP_VBUS
- R3 pad 1: FB_3V3 -> CP_VBUS
- R4 pad 2: EN -> FB_3V3
- R5 pad 1: +3V3 -> FB_3V3
- R5 pad 2: IO0 -> GND
- R6 pad 1: STATUS_LED -> +3V3
- R6 pad 2: LED_A -> EN
- U1 pad 12: IO0 -> (no net)
- U1 pad 16: (no net) -> STATUS_LED
- U1 pad 22: STATUS_LED -> IO8_STRAP
- U1 pad 23: (no net) -> BOOT
- U1 pad 5: (no net) -> IO2_STRAP
- U3 pad 8: VBUS -> CP_VBUS
Routing:
- net GND: track 117.5 -> 28.9 mm, vias 1 -> 26
- net BOOT: track 0.00 -> 13.9 mm, vias 0 -> 1
- net EN: track 11.7 -> 24.7 mm, vias 1 -> 2
- net IO0: track 12.1 -> 0.00 mm, vias 1 -> 0
- net STATUS_LED: track 12.9 -> 5.90 mm, vias 2 -> 0
- net CP_VBUS: track 0.00 -> 5.39 mm, vias 0 -> 1
- net +3V3: track 55.5 -> 59.9 mm
- net VBUS: track 23.0 -> 27.3 mm, vias 0 -> 1
- net FB_3V3: track 3.28 -> 7.05 mm
- net IO8_STRAP: track 0.00 -> 3.62 mm, vias 0 -> 1
- net IO2_STRAP: track 0.00 -> 2.42 mm, vias 0 -> 1
- net USB_DP: track 9.09 -> 11.3 mm
- net CALC_DM: track 12.8 -> 10.9 mm, vias 1 -> 0
- net VBUS_IN: track 9.02 -> 7.72 mm, vias 0 -> 1
- net USB_DM: track 9.05 -> 10.3 mm
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- added copper zone on In1.Cu, net GND
Other:
- board text added: "4:BOOT 3:EN"
- board text removed: "4:IO0 3:EN"
