File: v4/hardware/kicad/nlink-lite/nlink-lite.kicad_sch (KiCad schematic)
At the start: 25 parts, among them J1 USB_MiniB_PLUG_to_calc, J4 PROG_PADS_TC2030, SW1 PWR_SW, U1 ESP32-C3-MINI-1-N4, U3 CP2102N-A02-GQFN24, U4 TLV62569DBV, U5 USBLC6-2SC6

Commit message: Updated v4 pcb
Parts:
- J4: footprint Connector:Tag-Connect_TC2030-IDC-FP_2x03_P1.27mm_Vertical -> Connector_PinHeader_1.27mm:PinHeader_2x03_P1.27mm_Vertical_SMD
Changed lines of the file:
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@@
     (pin "4")
     (pin "5")
-    (instances (project "nlink-lite" (path "/64131837-4a1f-4de3-8334-4490d762c31b" (reference "J1") (unit 1))))
+    (instances (project "nlink-lite" (path "/20eb363d-eb86-43e6-9091-14d6a7b86412" (reference "J1") (unit 1))))
   )
   (global_label "VBUS_IN" (shape passive) (at 34.92 34.92 180) (effects (font (size 1.27 1.27)) (justify right)))
@@
     (pin "5")
     (pin "6")
-    (instances (project "nlink-lite" (path "/64131837-4a1f-4de3-8334-4490d762c31b" (reference "U5") (unit 1))))
+    (instances (project "nlink-lite" (path "/20eb363d-eb86-43e6-9091-14d6a7b86412" (reference "U5") (unit 1))))
   )
   (global_label "CALC_DM" (shape passive) (at 64.92 40 180) (effects (font (size 1.27 1.27)) (justify right)))
@@
     (pin "8")
     (pin "9")
-    (instances (project "nlink-lite" (path "/64131837-4a1f-4de3-8334-4490d762c31b" (reference "U3") (unit 1))))
+    (instances (project "nlink-lite" (path "/20eb363d-eb86-43e6-9091-14d6a7b86412" (reference "U3") (unit 1))))
   )
   (no_connect (at 122.7 39.92))
@@
     (pin "1")
     (pin "2")
-    (instances (project "nlink-lite" (path "/64131837-4a1f-4de3-8334-4490d762c31b" (reference "R1") (unit 1))))
+    (instances (project "nlink-lite" (path "/20eb363d-eb86-43e6-9091-14d6a7b86412" (reference "R1") (unit 1))))
   )
   (global_label "+3V3" (shape passive) (at 140 26.19 90) (effects (font (size 1.27 1.27)) (justify left)))
@@
     (pin "1")
     (pin "2")
-    (instances (project "nlink-lite" (path "/64131837-4a1f-4de3-8334-4490d762c31b" (reference "C1") (unit 1))))
+    (instances (project "nlink-lite" (path "/20eb363d-eb86-43e6-9091-14d6a7b86412" (reference "C1") (unit 1))))
   )
   (global_label "+3V3" (shape passive) (at 150 26.19 90) (effects (font (size 1.27 1.27)) (justify left)))
@@
     (pin "1")
     (pin "2")
-    (instances (project "nlink-lite" (path "/64131837-4a1f-4de3-8334-4490d762c31b" (reference "C2") (unit 1))))
+    (instances (project "nlink-lite" (path "/20eb363d-eb86-43e6-9091-14d6a7b86412" (reference "C2") (unit 1))))
   )
   (global_label "+3V3" (shape passive) (at 160 26.19 90) (effects (font (size 1.27 1.27)) (justify left)))
@@
     (pin "2")
     (pin "3")
-    (instances (project "nlink-lite" (path "/64131837-4a1f-4de3-8334-4490d762c31b" (reference "SW1") (unit 1))))
+    (instances (project "nlink-lite" (path "/20eb363d-eb86-43e6-9091-14d6a7b86412" (reference "SW1") (unit 1))))
   )
   (global_label "VBUS" (shape passive) (at 45.08 92.46 0) (effects (font (size 1.27 1.27)) (justify left)))
@@
     (pin "4")
     (pin "5")
-    (instances (project "nlink-lite" (path "/64131837-4a1f-4de3-8334-4490d762c31b" (reference "U4") (unit 1))))
+    (instances (project "nlink-lite" (path "/20eb363d-eb86-43e6-9091-14d6a7b86412" (reference "U4") (unit 1))))
   )
   (global_label "VBUS" (shape passive) (at 62.38 95 180) (effects (font (size 1.27 1.27)) (justify right)))
@@
     (pin "1")
     (pin "2")
-    (instances (project "nlink-lite" (path "/64131837-4a1f-4de3-8334-4490d762c31b" (reference "L1") (unit 1))))
+    (instances (project "nlink-lite" (path "/20eb363d-eb86-43e6-9091-14d6a7b86412" (reference "L1") (unit 1))))
   )
   (global_label "SW_NODE" (shape passive) (at 90 84.19 90) (effects (font (size 1.27 1.27)) (justify left)))
@@
     (pin "1")
     (pin "2")
-    (instances (project "nlink-lite" (path "/64131837-4a1f-4de3-8334-4490d762c31b" (reference "R2") (unit 1))))
+    (instances (project "nlink-lite" (path "/20eb363d-eb86-43e6-9091-14d6a7b86412" (reference "R2") (unit 1))))
   )
   (global_label "+3V3" (shape passive) (at 100 84.19 90) (effects (font (size 1.27 1.27)) (justify left)))
@@
     (pin "1")
     (pin "2")
-    (instances (project "nlink-lite" (path "/64131837-4a1f-4de3-8334-4490d762c31b" (reference "R3") (unit 1))))
+    (instances (project "nlink-lite" (path "/20eb363d-eb86-43e6-9091-14d6a7b86412" (reference "R3") (unit 1))))
   )
   (global_label "FB_3V3" (shape passive) (at 108 84.19 90) (effects (font (size 1.27 1.27)) (justify left)))
@@
     (pin "1")
     (pin "2")
-    (instances (project "nlink-lite" (path "/64131837-4a1f-4de3-8334-4490d762c31b" (reference "C3") (unit 1))))
+    (instances (project "nlink-lite" (path "/20eb363d-eb86-43e6-9091-14d6a7b86412" (reference "C3") (unit 1))))
   )
   (global_label "VBUS" (shape passive) (at 116 84.19 90) (effects (font (size 1.27 1.27)) (justify left)))
@@
     (pin "1")
     (pin "2")
-    (instances (project "nlink-lite" (path "/64131837-4a1f-4de3-8334-4490d762c31b" (reference "C4") (unit 1))))
+    (instances (project "nlink-lite" (path "/20eb363d-eb86-43e6-9091-14d6a7b86412" (reference "C4") (unit 1))))
   )
   (global_label "+3V3" (shape passive) (at 124 84.19 90) (effects (font (size 1.27 1.27)) (justify left)))
@@
     (pin "1")
     (pin "2")
-    (instances (project "nlink-lite" (path "/64131837-4a1f-4de3-8334-4490d762c31b" (reference "C5") (unit 1))))
+    (instances (project "nlink-lite" (path "/20eb363d-eb86-43e6-9091-14d6a7b86412" (reference "C5") (unit 1))))
   )
   (global_label "+3V3" (shape passive) (at 132 84.19 90) (effects (font (size 1.27 1.27)) (justify left)))
@@
     (pin "1")
     (pin "2")
-    (instances (project "nlink-lite" (path "/64131837-4a1f-4de3-8334-4490d762c31b" (reference "C6") (unit 1))))
+    (instances (project "nlink-lite" (path "/20eb363d-eb86-43e6-9091-14d6a7b86412" (reference "C6") (unit 1))))
   )
   (global_label "+3V3" (shape passive) (at 140 84.19 90) (effects (font (size 1.27 1.27)) (justify left)))
@@
     (pin "1")
     (pin "2")
-    (instances (project "nlink-lite" (path "/64131837-4a1f-4de3-8334-4490d762c31b" (reference "C7") (unit 1))))
+    (instances (project "nlink-lite" (path "/20eb363d-eb86-43e6-9091-14d6a7b86412" (reference "C7") (unit 1))))
   )
   (global_label "+3V3" (shape passive) (at 148 84.19 90) (effects (font (size 1.27 1.27)) (justify left)))
@@
     (property "Value" "PROG_PADS_TC2030" (at 150 100 0)
       (effects (font (size 1.27 1.27))))
-    (property "Footprint" "Connector:Tag-Connect_TC2030-IDC-FP_2x03_P1.27mm_Vertical" (at 150 100 0)
+    (property "Footprint" "Connector_PinHeader_1.27mm:PinHeader_2x03_P1.27mm_Vertical_SMD" (at 150 100 0)
       (effects (font (size 1.27 1.27)) hide))
     (property "Datasheet" "" (at 150 100 0)
@@
     (pin "5")
     (pin "6")
-    (instances (project "nlink-lite" (path "/64131837-4a1f-4de3-8334-4490d762c31b" (reference "J4") (unit 1))))
+    (instances (project "nlink-lite" (path "/20eb363d-eb86-43e6-9091-14d6a7b86412" (reference "J4") (unit 1))))
   )
   (global_label "+3V3" (shape passive) (at 144.92 94.92 180) (effects (font (size 1.27 1.27)) (justify right)))
@@
     (pin "1")
     (pin "2")
-    (instances (project "nlink-lite" (path "/64131837-4a1f-4de3-8334-4490d762c31b" (reference "R4") (unit 1))))
+    (instances (project "nlink-lite" (path "/20eb363d-eb86-43e6-9091-14d6a7b86412" (reference "R4") (unit 1))))
   )
   (global_label "+3V3" (shape passive) (at 175 88.19 90) (effects (font (size 1.27 1.27)) (justify left)))
@@
     (pin "1")
     (pin "2")
-    (instances (project "nlink-lite" (path "/64131837-4a1f-4de3-8334-4490d762c31b" (reference "C8") (unit 1))))
+    (instances (project "nlink-lite" (path "/20eb363d-eb86-43e6-9091-14d6a7b86412" (reference "C8") (unit 1))))
   )
   (global_label "EN" (shape passive) (at 183 88.19 90) (effects (font (size 1.27 1.27)) (justify left)))
@@
     (pin "1")
     (pin "2")
-    (instances (project "nlink-lite" (path "/64131837-4a1f-4de3-8334-4490d762c31b" (reference "R5") (unit 1))))
+    (instances (project "nlink-lite" (path "/20eb363d-eb86-43e6-9091-14d6a7b86412" (reference "R5") (unit 1))))
   )
   (global_label "+3V3" (shape passive) (at 191 88.19 90) (effects (font (size 1.27 1.27)) (justify left)))
@@
     (pin "1")
     (pin "2")
-    (instances (project "nlink-lite" (path "/64131837-4a1f-4de3-8334-4490d762c31b" (reference "R6") (unit 1))))
+    (instances (project "nlink-lite" (path "/20eb363d-eb86-43e6-9091-14d6a7b86412" (reference "R6") (unit 1))))
   )
   (global_label "STATUS_LED" (shape passive) (at 199 88.19 90) (effects (font (size 1.27 1.27)) (justify left)))
@@
     (pin "1")
     (pin "2")
-    (instances (project "nlink-lite" (path "/64131837-4a1f-4de3-8334-4490d762c31b" (reference "D1") (unit 1))))
+    (instances (project "nlink-lite" (path "/20eb363d-eb86-43e6-9091-14d6a7b86412" (reference "D1") (unit 1))))
   )
   (global_label "GND" (shape passive) (at 203.19 100 180) (effects (font (size 1.27 1.27)) (justify right)))
@@
     (pin "52")
     (pin "53")
-    (instances (project "nlink-lite" (path "/64131837-4a1f-4de3-8334-4490d762c31b" (reference "U1") (unit 1))))
+    (instances (project "nlink-lite" (path "/20eb363d-eb86-43e6-9091-14d6a7b86412" (reference "U1") (unit 1))))
   )
   (global_label "GND" (shape passive) (at 270 97.94 270) (effects (font (size 1.27 1.27)) (justify left)))
@@
     (pin "1")
     (pin "2")
-    (instances (project "nlink-lite" (path "/64131837-4a1f-4de3-8334-4490d762c31b" (reference "C9") (unit 1))))
+    (instances (project "nlink-lite" (path "/20eb363d-eb86-43e6-9091-14d6a7b86412" (reference "C9") (unit 1))))
   )
   (global_label "+3V3" (shape passive) (at 300 36.19 90) (effects (font (size 1.27 1.27)) (justify left)))
@@
     (pin "1")
     (pin "2")
-    (instances (project "nlink-lite" (path "/64131837-4a1f-4de3-8334-4490d762c31b" (reference "C10") (unit 1))))
+    (instances (project "nlink-lite" (path "/20eb363d-eb86-43e6-9091-14d6a7b86412" (reference "C10") (unit 1))))
   )
   (global_label "+3V3" (shape passive) (at 308 36.19 90) (effects (font (size 1.27 1.27)) (justify left)))

Commit message: Community caught bugs
Parts:
- removed C10: 10u, Capacitor_SMD:C_0805_2012Metric, symbol Device:C
- removed C8, C9: 100n, Capacitor_SMD:C_0402_1005Metric, symbol Device:C
- added R10, R7, R9: 10k, Resistor_SMD:R_0402_1005Metric, symbol Device:R
- added R8: 470, Resistor_SMD:R_0402_1005Metric, symbol Device:R
- C5: value 22u -> 100n; footprint Capacitor_SMD:C_0805_2012Metric -> Capacitor_SMD:C_0402_1005Metric
- C6: value 100u -> 100n; footprint Capacitor_SMD:C_1210_3225Metric -> Capacitor_SMD:C_0402_1005Metric
- C7: value 100u -> 10u; footprint Capacitor_SMD:C_1210_3225Metric -> Capacitor_SMD:C_0805_2012Metric
- J1: footprint (none) -> Connector_PinHeader_2.54mm:PinHeader_1x05_P2.54mm_Vertical
- R1: value 10k -> 1k
- R2: value 453k -> 22.1k
- R3: value 100k -> 47.5k
- R4: value 10k -> 453k
- R5: value 10k -> 100k
- R6: value 470 -> 10k
- SW1: footprint (none) -> Button_Switch_SMD:SW_SPDT_PCM12
Connections:
- net +3V3: now also R6.1, R10.1, R7.1, R9.1; no longer C5.1, R2.1, R5.1
- net EN: now also C5.1, R6.2; no longer R4.2
- net FB_3V3: now also R4.2, R5.1; no longer R2.2, R3.1
- net GND: now also J1.4 (Pin_4), R5.2
- net LED_A: now also R8.2; no longer R6.2
- net STATUS_LED: now also U1.16 (GPIO10), R8.1; no longer R6.1, U1.22 (GPIO8)
- net VBUS: now also R2.1; no longer U3.8 (VBUS)
- net BOOT: now reaches U1.23 (GPIO9)
- net BOOT: now also J4.4 (Pin_4), R7.2
- net IO2_STRAP: now reaches U1.5 (GPIO2/ADC1_CH2)
- net IO2_STRAP: now also R10.2
- removed net IO0: J4.4 (Pin_4), R5.2, U1.12 (GPIO0/ADC1_CH0/XTAL_32K_P)
- new net CP_VBUS: R2.2, R3.1, U3.8 (VBUS)
- new net IO8_STRAP: R9.2, U1.22 (GPIO8)
- no-connect marks 39 -> 36
Other:
- note added: "PROGRAM — TC2030/pogo: USB + straps (GPIO9 low at boot = flash)"
- note added: "lite: TLV62569 Cout 10-47uF - no 100uF bulk"
- note removed: "PROGRAM — TC2030/pogo: USB + straps (IO0 low at boot = flash)"
